File: hardware/hardware-puck-carrier/puck-carrier.kicad_pcb (KiCad board)
At the start: 4 copper layers, 46 x 46 mm, 124 parts, among them J1 LiPo 400-500mAh protected, Q1 AO3400A, Q2 AO3400A, Q3 AO3400A, Q4 AO3400A, Q5 AO3400A, U1 MDBT50Q-1MV2, U10 XC6206P182MR 1.8V->AS7341 only, U11 USBLC6-2SC6, U2 TPS61023, U3 AS7341, U4 FDC1004, U5 MS5837-02BA, U6 DS18B20U+, U7 MCP73832T-2ACI/OT, U8 LSM6DSO, U9 IM69D130

Commit message: Round PCB traces and repair USB, battery and 3V3 connections
Preserve the original full-feature layout. Verify zero DRC violations and schematic mismatches, with 21 opens still outstanding; this is not a fabrication release. Fix raster connectivity and project-aware geometry export, and refresh reports and previews.
Routing:
- net VBAT: track 60.9 -> 75.1 mm, vias 3 -> 4
- net GND: track 152.5 -> 161.4 mm, vias 38 -> 45
- net EC_SENSE_B: track 4.32 -> 2.49 mm, vias 3 -> 1
- net VBUS: track 29.0 -> 30.7 mm, vias 0 -> 2
- net EC_SENSE_A: track 5.52 -> 4.09 mm, vias 2 -> 1
- net /PAD_DM: track 14.2 -> 15.4 mm
- net IMU_INT: track 0.90 -> 0.00 mm, vias 1 -> 0
- net CHG_STAT: track 0.90 -> 0.00 mm, vias 1 -> 0
- net SHLD1: track 13.1 -> 12.4 mm
- net RESET: track 33.7 -> 33.5 mm, vias 3 -> 2
- net 3V3: track 134.4 -> 134.6 mm, vias 23 -> 24
- net RING_DATA: track 19.1 -> 19.0 mm, vias 1 -> 0
