File: hardware/hardware-puck-carrier/puck-carrier.kicad_pcb (KiCad board)
At the start: 4 copper layers, 46 x 46 mm, 124 parts, among them J1 LiPo 400-500mAh protected, Q1 AO3400A, Q2 AO3400A, Q3 AO3400A, Q4 AO3400A, Q5 AO3400A, U1 MDBT50Q-1MV2, U10 XC6206P182MR 1.8V->AS7341 only, U11 USBLC6-2SC6, U2 TPS61023, U3 AS7341, U4 FDC1004, U5 MS5837-02BA, U6 DS18B20U+, U7 MCP73832T-2ACI/OT, U8 LSM6DSO, U9 IM69D130

Commit message: Checkpoint before archive cleanup: v2 board, routes, research notes, pin-swap variant
Co-Authored-By: Claude Fable 5.1 <noreply@anthropic.com>
Routing:
- net GND: track 161.4 -> 164.4 mm, vias 45 -> 44
- net RESET: track 33.5 -> 36.0 mm
- net VBAT: track 75.1 -> 75.8 mm
